File: calc-project.kicad_pcb (KiCad board)
At the start: 2 copper layers, 80 x 100 mm, 46 parts, among them J1 PinSocket_1x20_Right, J2 PinSocket_1x20_Left, J3 Conn_01x14, SW1 SW_Push_45deg, SW10 SW_Push_45deg, SW11 SW_Push_45deg, SW12 SW_Push_45deg, SW13 SW_Push_45deg, SW14 SW_Push_45deg, SW15 SW_Push_45deg, SW16 SW_Push_45deg, SW17 SW_Push_45deg, SW18 SW_Push_45deg, SW19 SW_Push_45deg, SW2 SW_Push_45deg, SW20 SW_Push_45deg, SW21 SW_Push_45deg, SW22 SW_Push_45deg, SW23 SW_Push_45deg, SW24 SW_Push_45deg, SW25 SW_Push_45deg, SW26 SW_Push_45deg, SW27 SW_Push_45deg, SW28 SW_Push_45deg, SW29 SW_Push_45deg, SW3 SW_Push_45deg, SW30 SW_Push_45deg, SW31 SW_Push_45deg, SW32 SW_Push_45deg, SW33 SW_Push_45deg, SW34 SW_Push_45deg, SW35 SW_Push_45deg, SW36 SW_Push_45deg, SW4 SW_Push_45deg, SW5 SW_Push_45deg, SW6 SW_Push_45deg, SW7 SW_Push_45deg, SW8 SW_Push_45deg, SW9 SW_Push_45deg

Commit message: mb one last connection
Routing:
- net row 0: track 68.8 -> 74.3 mm
Changed lines of the file:
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@@
+	)
+	(segment
+		(start 53.25 112.25)
+		(end 58.75 112.25)
+		(width 0.2)
+		(layer "F.Cu")
+		(net "row 0")
 	)
 	(segment
